File: Electronic_design/STM32_PAP_board/STM32&PAP_board.brd (EAGLE design)
At the start: 100 x 80 mm, 20 parts

Commit message: reroutage carte IMU et STEPPER
Parts:
- removed U$5: AUTO_FUSE, AUTO_FUSE:AUTO_FUSE
- added F1: (no value), fuse:TR5
- added SL1: (no value), con-amp-quick:03P
Connections:
- net 3V: now also F1.2; no longer U$5.P$4
- net GND: now also SL1.3
- net N$13: now also SL1.1
- net N$14: now also SL1.2
- net N$41: now also F1.1; no longer U$5.P$2
Routing:
- net GND: track 59.1 -> 0.61 mm
- net N$42: track 63.6 -> 27.8 mm
- net N$13: track 5.15 -> 40.7 mm
- net N$14: track 5.24 -> 34.3 mm
- net N$41: track 13.2 -> 16.7 mm
- net 3V: track 130.1 -> 133.0 mm
