File: Electronic_design/STM32_PAP_board/STM32&PAP_board.sch (EAGLE design)
At the start: 20 parts

Commit message: reroutage carte IMU et STEPPER
Parts:
- removed U$5: AUTO_FUSE, AUTO_FUSE:AUTO_FUSE
- added F1: (no value), fuse:TR5
- added SL1: (no value), con-amp-quick:MA03
Connections:
- net 3V: now also F1.2; no longer U$5.P$2
- net GND: now also SL1.3
- net N$13: now also SL1.1
- net N$14: now also SL1.2
- net N$41: now also F1.1; no longer U$5.P$1
Changed lines of the file:
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@@
 <?xml version="1.0" encoding="utf-8"?>
 <!DOCTYPE eagle SYSTEM "eagle.dtd">
-<eagle version="8.4.1">
+<eagle version="6.5.0">
 <drawing>
 <settings>
@@
 <part name="U$3" library="stm32duino boards" deviceset="BLUEPILL" device=""/>
 <part name="U$4" library="AUTO_FUSE" deviceset="AUTO_FUSE" device=""/>
-<part name="SV1" library="con-lstb" library_urn="urn:adsk.eagle:library:162" deviceset="MA03-1" device="" package3d_urn="urn:adsk.eagle:package:8339/1"/>
-<part name="SV2" library="con-lstb" library_urn="urn:adsk.eagle:library:162" deviceset="MA20-1" device="" package3d_urn="urn:adsk.eagle:package:8359/1"/>
-<part name="SV3" library="con-lstb" library_urn="urn:adsk.eagle:library:162" deviceset="MA20-1" device="" package3d_urn="urn:adsk.eagle:package:8359/1"/>
-<part name="3.3V" library="v-reg" library_urn="urn:adsk.eagle:library:409" deviceset="LM138-TS" device="" package3d_urn="urn:adsk.eagle:package:30366/1"/>
-<part name="U$5" library="AUTO_FUSE" deviceset="AUTO_FUSE" device=""/>
-<part name="SV4" library="con-lstb" library_urn="urn:adsk.eagle:library:162" deviceset="MA04-1" device="" package3d_urn="urn:adsk.eagle:package:8337/1"/>
-<part name="SV5" library="con-lstb" library_urn="urn:adsk.eagle:library:162" deviceset="MA04-1" device="" package3d_urn="urn:adsk.eagle:package:8337/1"/>
-<part name="ALIM_3V" library="con-molex" library_urn="urn:adsk.eagle:library:165" deviceset="22-?-02" device="27-2021"/>
-<part name="SV6" library="con-lstb" library_urn="urn:adsk.eagle:library:162" deviceset="MA06-2" device="" package3d_urn="urn:adsk.eagle:package:8342/1"/>
-<part name="SV7" library="con-lstb" library_urn="urn:adsk.eagle:library:162" deviceset="MA06-2" device="" package3d_urn="urn:adsk.eagle:package:8342/1"/>
-<part name="SV8" library="con-lstb" library_urn="urn:adsk.eagle:library:162" deviceset="MA10-2" device="" package3d_urn="urn:adsk.eagle:package:8331/1"/>
-<part name="SV9" library="con-lstb" library_urn="urn:adsk.eagle:library:162" deviceset="MA10-2" device="" package3d_urn="urn:adsk.eagle:package:8331/1"/>
-<part name="SV10" library="con-lstb" library_urn="urn:adsk.eagle:library:162" deviceset="MA10-2" device="" package3d_urn="urn:adsk.eagle:package:8331/1"/>
-<part name="SV11" library="con-lstb" library_urn="urn:adsk.eagle:library:162" deviceset="MA10-2" device="" package3d_urn="urn:adsk.eagle:package:8331/1"/>
-<part name="C1" library="capacitor-wima" library_urn="urn:adsk.eagle:library:116" deviceset="C" device="5/5" package3d_urn="urn:adsk.eagle:package:5428/1"/>
-<part name="C2" library="capacitor-wima" library_urn="urn:adsk.eagle:library:116" deviceset="C" device="5/5" package3d_urn="urn:adsk.eagle:package:5428/1"/>
+<part name="SV1" library="con-lstb" deviceset="MA03-1" device=""/>
+<part name="SV2" library="con-lstb" deviceset="MA20-1" device=""/>
+<part name="SV3" library="con-lstb" deviceset="MA20-1" device=""/>
+<part name="3.3V" library="v-reg" deviceset="LM138-TS" device=""/>
+<part name="SV4" library="con-lstb" deviceset="MA04-1" device=""/>
+<part name="SV5" library="con-lstb" deviceset="MA04-1" device=""/>
+<part name="ALIM_3V" library="con-molex" deviceset="22-?-02" device="27-2021"/>
+<part name="SV6" library="con-lstb" deviceset="MA06-2" device=""/>
+<part name="SV7" library="con-lstb" deviceset="MA06-2" device=""/>
+<part name="SV8" library="con-lstb" deviceset="MA10-2" device=""/>
+<part name="SV9" library="con-lstb" deviceset="MA10-2" device=""/>
+<part name="SV10" library="con-lstb" deviceset="MA10-2" device=""/>
+<part name="SV11" library="con-lstb" deviceset="MA10-2" device=""/>
+<part name="C1" library="capacitor-wima" deviceset="C" device="5/5"/>
+<part name="C2" library="capacitor-wima" deviceset="C" device="5/5"/>
+<part name="F1" library="fuse" deviceset="TR5" device=""/>
+<part name="SL1" library="con-amp-quick" deviceset="MA03" device=""/>
 </parts>
 <sheets>
@@
 <instance part="SV3" gate="1" x="-5.08" y="7.62" rot="R180"/>
 <instance part="3.3V" gate="G$1" x="-17.78" y="50.8"/>
-<instance part="U$5" gate="G$1" x="5.08" y="50.8"/>
 <instance part="SV4" gate="1" x="124.46" y="20.32" rot="R180"/>
 <instance part="SV5" gate="1" x="124.46" y="-15.24" rot="R180"/>
@@
 <instance part="C1" gate="G$1" x="35.56" y="58.42"/>
 <instance part="C2" gate="G$1" x="44.45" y="58.42"/>
+<instance part="F1" gate="1" x="5.08" y="50.8"/>
+<instance part="SL1" gate="G$1" x="-99.06" y="15.24"/>
 </instances>
 <busses>
@@
 <pinref part="SV2" gate="1" pin="13"/>
 <wire x1="-73.66" y1="12.7" x2="-63.5" y2="12.7" width="0.1524" layer="91"/>
+<pinref part="SL1" gate="G$1" pin="1"/>
+<wire x1="-91.44" y1="12.7" x2="-73.66" y2="12.7" width="0.1524" layer="91"/>
 </segment>
 </net>
@@
 <pinref part="SV2" gate="1" pin="14"/>
 <wire x1="-73.66" y1="15.24" x2="-63.5" y2="15.24" width="0.1524" layer="91"/>
+<pinref part="SL1" gate="G$1" pin="2"/>
+<wire x1="-91.44" y1="15.24" x2="-73.66" y2="15.24" width="0.1524" layer="91"/>
 </segment>
 </net>
@@
 <label x="35.56" y="53.34" size="1.778" layer="95" rot="R180"/>
 </segment>
+<segment>
+<pinref part="SL1" gate="G$1" pin="3"/>
+<wire x1="-91.44" y1="17.78" x2="-86.36" y2="17.78" width="0.1524" layer="91"/>
+<label x="-91.44" y="17.78" size="1.778" layer="95"/>
+</segment>
 </net>
 <net name="N$43" class="0">
@@
 <segment>
 <pinref part="3.3V" gate="G$1" pin="OUT"/>
-<pinref part="U$5" gate="G$1" pin="P$1"/>
-<wire x1="-10.16" y1="50.8" x2="-5.08" y2="50.8" width="0.1524" layer="91"/>
+<pinref part="F1" gate="1" pin="1"/>
+<wire x1="-10.16" y1="50.8" x2="0" y2="50.8" width="0.1524" layer="91"/>
 </segment>
 </net>
@@
 <net name="3V" class="0">
 <segment>
-<pinref part="U$5" gate="G$1" pin="P$2"/>
-<junction x="17.78" y="50.8"/>
 <label x="20.32" y="50.8" size="1.778" layer="95"/>
 <wire x1="20.32" y1="50.8" x2="17.78" y2="50.8" width="0.1524" layer="91"/>
@@
 <wire x1="76.2" y1="40.64" x2="76.2" y2="15.24" width="0.1524" layer="91"/>
 <wire x1="76.2" y1="15.24" x2="86.36" y2="15.24" width="0.1524" layer="91"/>
+<pinref part="F1" gate="1" pin="2"/>
+<wire x1="10.16" y1="50.8" x2="17.78" y2="50.8" width="0.1524" layer="91"/>
+<junction x="17.78" y="50.8"/>
 </segment>
 <segment>
@@
 </schematic>
 </drawing>
-<compatibility>
-<note version="8.2" severity="warning">
-Since Version 8.2, EAGLE supports online libraries. The ids
-of those online libraries will not be understood (or retained)
-with this version.
-</note>
-<note version="8.3" severity="warning">
-Since Version 8.3, EAGLE supports URNs for individual library
-assets (packages, symbols, and devices). The URNs of those assets
-will not be understood (or retained) with this version.
-</note>
-<note version="8.3" severity="warning">
-Since Version 8.3, EAGLE supports the association of 3D packages
-with devices in libraries, schematics, and board files. Those 3D
-packages will not be understood (or retained) with this version.
-</note>
-</compatibility>
 </eagle>
