File: Electronic_design/IMU_adaptator/IMU_adaptator.brd (EAGLE design)
At the start: 47.7 x 34.1 mm, 6 parts, among them J1 CLM-110-02-XX-D

Commit message: ajout alim aux connect SPI et UART
Parts:
- removed SL1: (no value), con-amp-quick:05PA
- removed SL2: (no value), con-amp-quick:03P
- added SV2: (no value), con-lstb:MA06-1
- added SV3: (no value), con-lstb:MA04-1
- added SV4: (no value), con-lsta:FE06
Connections:
- new net SCK/TX: SV2.2
- net GND: now also SV2.6, SV3.4; no longer SL1.5, SL2.3
- net MISO/RX: now also SV2.3, SV3.2; no longer SL1.1, SL2.1
- net MOSI: now also SV2.4; no longer SL1.2
- net SLCK/TX: now also SV3.1; no longer SL1.3, SL2.2
- net SS: now also SV2.1; no longer SL1.4
- net VCC: now also SV2.5, SV3.3
Routing:
- net VCC: track 67.2 -> 103.3 mm
- net SLCK/TX: track 80.1 -> 65.0 mm, vias 3 -> 1
- net MISO/RX: track 74.7 -> 81.1 mm
- net MOSI: track 61.5 -> 61.6 mm, vias 3 -> 2

Commit message: suppression connecteur inutile
Parts:
- removed SV4: (no value), con-lsta:FE06
Changed lines of the file:
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@@
 <attribute name="OC_NEWARK" value="unknown" x="17" y="5" size="1.778" layer="27" display="off"/>
-</element>
-<element name="SV4" library="con-lsta" library_urn="urn:adsk.eagle:library:161" package="FE06" package3d_urn="urn:adsk.eagle:package:8191/1" value="" x="8.5" y="-40.5">
-<attribute name="MF" value="" x="8.5" y="-40.5" size="1.778" layer="27" display="off"/>
-<attribute name="MPN" value="" x="8.5" y="-40.5" size="1.778" layer="27" display="off"/>
-<attribute name="OC_FARNELL" value="unknown" x="8.5" y="-40.5" size="1.778" layer="27" display="off"/>
-<attribute name="OC_NEWARK" value="unknown" x="8.5" y="-40.5" size="1.778" layer="27" display="off"/>
 </element>
 </elements>
