File: Electronic_design/IMU_adaptator/IMU_adaptator.brd (EAGLE design)
At the start: 47.7 x 34.1 mm, 6 parts, among them J1 CLM-110-02-XX-D

Commit message: ajout LED
Parts:
- added R1: (no value), rcl:0204/5
- added VCC: (no value), eagle-ltspice:LED_LD260
Connections:
- new net N$7: R1.2, VCC.A
- net GND: now also VCC.K
- net VCC: now also R1.1
Routing:
- net VCC: track 103.3 -> 113.6 mm
- net N$7: track 0.00 -> 4.88 mm
Changed lines of the file:
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@@
 <text x="1.397" y="28.829" size="0.6096" layer="37" font="vector" rot="R180">4</text>
 <text x="7.366" y="28.448" size="0.6096" layer="37" font="vector" rot="R180">3</text>
-<text x="9.652" y="3.175" size="1.016" layer="25" font="vector" rot="R180">LAAS CNRS</text>
+<text x="9.152" y="33.175" size="1.016" layer="25" font="vector" rot="R180">LAAS CNRS</text>
 <text x="38.164" y="1.143" size="0.6096" layer="25" font="vector" rot="R90">GND</text>
 <text x="21.164" y="1.143" size="0.6096" layer="25" font="vector" rot="R90">GND</text>
@@
 <attribute name="VALUE" x="17.635" y="6.651" size="1.27" layer="27" ratio="10"/>
 </element>
+<element name="R1" library="rcl" library_urn="urn:adsk.eagle:library:334" package="0204/5" package3d_urn="urn:adsk.eagle:package:23488/1" value="" x="8.5" y="4" rot="R90"/>
+<element name="VCC" library="eagle-ltspice" library_urn="urn:adsk.eagle:library:217" package="LED_LD260" package3d_urn="urn:adsk.eagle:package:13313/1" value="" x="4" y="3" rot="R180">
+<attribute name="SPICEMODEL" value="NONE" x="4" y="3" size="1.778" layer="27" rot="R180" display="off"/>
+<attribute name="SPICEPREFIX" value="D" x="4" y="3" size="1.778" layer="27" rot="R180" display="off"/>
+<attribute name="SPICETYPE" value="diode" x="4" y="3" size="1.778" layer="27" rot="R180" display="off"/>
+</element>
 </elements>
 <signals>
@@
 <contactref element="SV2" pad="6"/>
 <contactref element="SV3" pad="4"/>
+<contactref element="VCC" pad="K"/>
 </signal>
 <signal name="N$13">
@@
 <wire x1="35.5" y1="3" x2="34" y2="1.5" width="0.6096" layer="1"/>
 <wire x1="34" y1="1.5" x2="19.5" y2="1.5" width="0.6096" layer="1"/>
-<wire x1="19.5" y1="1.5" x2="18.27" y2="2.73" width="0.6096" layer="1"/>
+<wire x1="18.27" y1="2.73" x2="19.5" y2="1.5" width="0.6096" layer="1"/>
 <wire x1="18.27" y1="2.73" x2="18.27" y2="5" width="0.6096" layer="1"/>
+<contactref element="R1" pad="1"/>
+<wire x1="8.5" y1="1.46" x2="17" y2="1.46" width="0.508" layer="1"/>
+<wire x1="17" y1="1.46" x2="18.27" y2="2.73" width="0.508" layer="1"/>
 </signal>
 <signal name="SLCK/TX">
@@
 <contactref element="SV2" pad="2"/>
 </signal>
+<signal name="N$7">
+<contactref element="R1" pad="2"/>
+<contactref element="VCC" pad="A"/>
+<wire x1="5.27" y1="3" x2="8.5" y2="6.23" width="0.508" layer="1"/>
+<wire x1="8.5" y1="6.23" x2="8.5" y2="6.54" width="0.508" layer="1"/>
+</signal>
 </signals>

Commit message: nouveau routage
Parts:
- moved SV1 0.71 mm to (4.31, 19.6), turned to 90 degrees
- turned J1 to 90 degrees
Connections:
- net N$1 renamed 1
- net N$2 renamed 2
- net N$20 renamed 20
- net SCK/TX: now also J1.3, SV1.3
- net SLCK/TX: no longer J1.3, SV1.3
Routing:
- net SLCK/TX: track 65.0 -> 0.00 mm, vias 1 -> 0
- net SCK/TX: track 0.00 -> 48.3 mm, vias 0 -> 2
- net MISO/RX: track 81.1 -> 59.2 mm
- net SS: track 59.8 -> 52.1 mm, vias 1 -> 2
- net N$14: track 45.8 -> 41.2 mm, vias 2 -> 0
- net N$13: track 44.0 -> 40.6 mm, vias 2 -> 0
- net MOSI: track 61.6 -> 64.8 mm
- net 2: track 41.5 -> 44.7 mm
- net N$23: track 44.5 -> 42.4 mm
- net VCC: track 113.6 -> 112.3 mm, vias 0 -> 1
- net N$22: track 44.3 -> 43.0 mm
- net 20: track 44.4 -> 43.2 mm, vias 2 -> 0
- net N$18: track 41.3 -> 42.1 mm, vias 0 -> 2
- net N$9: track 41.5 -> 40.8 mm, vias 2 -> 1
- net N$8: track 40.8 -> 41.6 mm, vias 2 -> 0
Other:
- board text removed: "2"
- board text removed: "3"
- board text removed: "4"
