File: Electronic_design/PowerBoard/Power.Board.sch (EAGLE design)
At the start: 32 parts, among them IC1 788TV, IC2 788TV

Commit message: ajout condensateurs
Parts:
- added C1, C2, C3: (no value), rcl:CPOL-EUE7.5-18
- added C4: (no value), rcl:CPOL-EUE5-13
Connections:
- net 12V: now also C1.+, C2.+, C3.+
- net GND: now also C1.-, C2.-, C3.-, C4.-
- net N$6: now also C4.+
Other:
- moved on the sheet: U$5
Changed lines of the file:
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@@
 <part name="LED6" library="eagle-ltspice" library_urn="urn:adsk.eagle:library:217" deviceset="LED_E" device="LD260" package3d_urn="urn:adsk.eagle:package:13313/1"/>
 <part name="IC2" library="linear" library_urn="urn:adsk.eagle:library:262" deviceset="78*" device="TV" package3d_urn="urn:adsk.eagle:package:16417/1" technology="8"/>
+<part name="C1" library="rcl" library_urn="urn:adsk.eagle:library:334" deviceset="CPOL-EU" device="E7.5-18" package3d_urn="urn:adsk.eagle:package:23379/1"/>
+<part name="C2" library="rcl" library_urn="urn:adsk.eagle:library:334" deviceset="CPOL-EU" device="E7.5-18" package3d_urn="urn:adsk.eagle:package:23379/1"/>
+<part name="C3" library="rcl" library_urn="urn:adsk.eagle:library:334" deviceset="CPOL-EU" device="E7.5-18" package3d_urn="urn:adsk.eagle:package:23379/1"/>
+<part name="C4" library="rcl" library_urn="urn:adsk.eagle:library:334" deviceset="CPOL-EU" device="E5-13" package3d_urn="urn:adsk.eagle:package:23375/1"/>
 </parts>
 <sheets>
@@
 <instance part="MAST1" gate="G$1" x="5.08" y="-25.4"/>
 <instance part="PAP1" gate="G$1" x="5.08" y="-40.64"/>
-<instance part="U$5" gate="G$1" x="-48.26" y="-12.7" rot="R90"/>
+<instance part="U$5" gate="G$1" x="-66.04" y="-12.7" rot="R90"/>
 <instance part="0D2" gate="G$1" x="33.02" y="-10.16"/>
 <instance part="MAST2" gate="G$1" x="33.02" y="-25.4"/>
@@
 <instance part="LED6" gate="G$1" x="71.12" y="-106.68" rot="R90"/>
 <instance part="IC2" gate="A1" x="33.02" y="-96.52"/>
+<instance part="C1" gate="G$1" x="-30.48" y="-20.32"/>
+<instance part="C2" gate="G$1" x="-22.86" y="-20.32"/>
+<instance part="C3" gate="G$1" x="-15.24" y="-20.32"/>
+<instance part="C4" gate="G$1" x="48.26" y="-12.7"/>
 </instances>
 <busses>
@@
 <wire x1="-5.08" y1="-78.74" x2="-5.08" y2="-55.88" width="0.1524" layer="91"/>
 <wire x1="-5.08" y1="-55.88" x2="-5.08" y2="-40.64" width="0.1524" layer="91"/>
-<wire x1="-43.18" y1="-10.16" x2="-5.08" y2="-10.16" width="0.1524" layer="91"/>
+<wire x1="-60.96" y1="-10.16" x2="-15.24" y2="-10.16" width="0.1524" layer="91"/>
 <junction x="-5.08" y="-10.16"/>
 <pinref part="RPI" gate="G$1" pin="1A"/>
+<wire x1="-15.24" y1="-10.16" x2="-5.08" y2="-10.16" width="0.1524" layer="91"/>
 <wire x1="2.54" y1="-78.74" x2="-5.08" y2="-78.74" width="0.1524" layer="91"/>
 <junction x="-5.08" y="-78.74"/>
 <pinref part="FNU1" gate="G$1" pin="P$1"/>
 <junction x="-5.08" y="-55.88"/>
+<pinref part="C1" gate="G$1" pin="+"/>
+<pinref part="C2" gate="G$1" pin="+"/>
+<wire x1="-30.48" y1="-17.78" x2="-22.86" y2="-17.78" width="0.1524" layer="91"/>
+<pinref part="C3" gate="G$1" pin="+"/>
+<wire x1="-22.86" y1="-17.78" x2="-15.24" y2="-17.78" width="0.1524" layer="91"/>
+<junction x="-22.86" y="-17.78"/>
+<wire x1="-15.24" y1="-17.78" x2="-15.24" y2="-10.16" width="0.1524" layer="91"/>
+<junction x="-15.24" y="-17.78"/>
+<junction x="-15.24" y="-10.16"/>
 </segment>
 </net>
@@
 <pinref part="0D2" gate="G$1" pin="P$2"/>
 <pinref part="OD" gate="G$1" pin="P$1"/>
-<wire x1="45.72" y1="-10.16" x2="55.88" y2="-10.16" width="0.1524" layer="91"/>
+<wire x1="45.72" y1="-10.16" x2="48.26" y2="-10.16" width="0.1524" layer="91"/>
 <pinref part="R1" gate="G$1" pin="1"/>
+<wire x1="48.26" y1="-10.16" x2="55.88" y2="-10.16" width="0.1524" layer="91"/>
 <wire x1="55.88" y1="-10.16" x2="86.36" y2="-10.16" width="0.1524" layer="91"/>
 <wire x1="55.88" y1="-20.32" x2="55.88" y2="-10.16" width="0.1524" layer="91"/>
 <junction x="55.88" y="-10.16"/>
+<pinref part="C4" gate="G$1" pin="+"/>
+<junction x="48.26" y="-10.16"/>
 </segment>
 </net>
@@
 <wire x1="101.6" y1="-12.7" x2="101.6" y2="-25.4" width="0.1524" layer="91"/>
 <pinref part="U$5" gate="G$1" pin="P$1"/>
-<wire x1="-43.18" y1="-15.24" x2="-43.18" y2="-114.3" width="0.1524" layer="91"/>
-<wire x1="-43.18" y1="-114.3" x2="33.02" y2="-114.3" width="0.1524" layer="91"/>
-<wire x1="33.02" y1="-114.3" x2="101.6" y2="-114.3" width="0.1524" layer="91"/>
+<wire x1="-60.96" y1="-15.24" x2="-60.96" y2="-25.4" width="0.1524" layer="91"/>
+<wire x1="-60.96" y1="-25.4" x2="-60.96" y2="-114.3" width="0.1524" layer="91"/>
+<wire x1="-60.96" y1="-114.3" x2="15.24" y2="-114.3" width="0.1524" layer="91"/>
+<wire x1="15.24" y1="-114.3" x2="101.6" y2="-114.3" width="0.1524" layer="91"/>
 <wire x1="101.6" y1="-114.3" x2="101.6" y2="-106.68" width="0.1524" layer="91"/>
 <wire x1="101.6" y1="-106.68" x2="101.6" y2="-101.6" width="0.1524" layer="91"/>
@@
 <junction x="101.6" y="-106.68"/>
 <pinref part="IC2" gate="A1" pin="GND"/>
-<wire x1="33.02" y1="-104.14" x2="33.02" y2="-114.3" width="0.1524" layer="91"/>
-<junction x="33.02" y="-114.3"/>
-</segment>
-<segment>
+<wire x1="33.02" y1="-104.14" x2="15.24" y2="-114.3" width="0.1524" layer="91"/>
+<junction x="15.24" y="-114.3"/>
+<pinref part="C3" gate="G$1" pin="-"/>
+<pinref part="C2" gate="G$1" pin="-"/>
+<pinref part="C1" gate="G$1" pin="-"/>
+<wire x1="-30.48" y1="-25.4" x2="-22.86" y2="-25.4" width="0.1524" layer="91"/>
+<junction x="-22.86" y="-25.4"/>
+<wire x1="-22.86" y1="-25.4" x2="-15.24" y2="-25.4" width="0.1524" layer="91"/>
+<wire x1="-22.86" y1="-25.4" x2="-60.96" y2="-25.4" width="0.1524" layer="91"/>
+<junction x="-60.96" y="-25.4"/>
+<pinref part="C4" gate="G$1" pin="-"/>
+<wire x1="48.26" y1="-17.78" x2="48.26" y2="-22.86" width="0.1524" layer="91"/>
+<wire x1="48.26" y1="-22.86" x2="76.2" y2="-22.86" width="0.1524" layer="91"/>
+<wire x1="76.2" y1="-22.86" x2="76.2" y2="-20.32" width="0.1524" layer="91"/>
+<junction x="76.2" y="-20.32"/>
+</segment>
+<segment>
